File: KiCad/TankIR_Breaker/TankIR_Breaker.kicad_pcb (KiCad board)
At the start: 2 copper layers, 44.6 x 18.2 mm, 16 parts, among them J1 VBATT, J2 TRIGGER, J3 SERVO, J4 RC, J5 APPLE, J6 SOUND, J7 IR_OUT, J8 MUZZLE, Q1 BC337, Q2 BC337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

Commit message: change
Parts:
- moved J1 2.18 mm to (86.5, 69.0), turned to 0 degrees
Connections:
- J1 pad 1: GND -> +BATT
- J1 pad 2: +BATT -> GND
Other:
- board text added: "+"
- board text added: "S"
- board text added: "SERVO"
Changed lines of the file:
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@@
 			(outputformat 1)
 			(mirror no)
-			(drillshape 1)
+			(drillshape 0)
 			(scaleselection 1)
-			(outputdirectory "")
+			(outputdirectory "Gerber/")
 		)
 	)
@@
 	(footprint "Connector_JST:JST_PH_B2B-PH-K_1x02_P2.00mm_Vertical"
 		(layer "F.Cu")
-		(at 88.6 69.6 180)
+		(at 86.5 69)
 		(descr "JST PH series connector, B2B-PH-K (http://www.jst-mfg.com/product/pdf/eng/ePH.pdf), generated with kicad-footprint-generator")
 		(tags "connector JST PH vertical")
@@
 		(attr through_hole)
 		(fp_line
-			(start 4.06 2.91)
-			(end 4.06 -1.81)
+			(start -2.36 -2.11)
+			(end -2.36 -0.86)
 			(stroke
 				(width 0.12)
@@
 		)
 		(fp_line
-			(start 4.06 0.8)
-			(end 3.45 0.8)
+			(start -2.06 -1.81)
+			(end -2.06 2.91)
 			(stroke
 				(width 0.12)
@@
 		)
 		(fp_line
-			(start 4.06 -0.5)
-			(end 3.45 -0.5)
+			(start -2.06 -0.5)
+			(end -1.45 -0.5)
 			(stroke
 				(width 0.12)
@@
 		)
 		(fp_line
-			(start 4.06 -1.81)
-			(end -2.06 -1.81)
+			(start -2.06 0.8)
+			(end -1.45 0.8)
 			(stroke
 				(width 0.12)
@@
 		)
 		(fp_line
-			(start 3.45 2.3)
-			(end 3.45 -1.2)
+			(start -2.06 2.91)
+			(end 4.06 2.91)
 			(stroke
 				(width 0.12)
@@
 		)
 		(fp_line
-			(start 3.45 -1.2)
-			(end 1.5 -1.2)
+			(start -1.45 -1.2)
+			(end -1.45 2.3)
 			(stroke
 				(width 0.12)
@@
 		)
 		(fp_line
-			(start 1.5 -1.2)
-			(end 1.5 -1.81)
+			(start -1.45 2.3)
+			(end 3.45 2.3)
 			(stroke
 				(width 0.12)
@@
 		)
 		(fp_line
-			(start 1.1 1.8)
-			(end 1.1 2.3)
+			(start -1.11 -2.11)
+			(end -2.36 -2.11)
 			(stroke
 				(width 0.12)
@@
 		)
 		(fp_line
-			(start 1 2.3)
-			(end 1 1.8)
+			(start -0.6 -2.01)
+			(end -0.6 -1.81)
 			(stroke
 				(width 0.12)
@@
 		)
 		(fp_line
-			(start 0.9 2.3)
-			(end 0.9 1.8)
+			(start -0.3 -2.01)
+			(end -0.6 -2.01)
 			(stroke
 				(width 0.12)
@@
 		)
 		(fp_line
-			(start 0.9 1.8)
-			(end 1.1 1.8)
+			(start -0.3 -1.91)
+			(end -0.6 -1.91)
 			(stroke
 				(width 0.12)
@@
 		)
 		(fp_line
-			(start 0.5 -1.2)
-			(end -1.45 -1.2)
+			(start -0.3 -1.81)
+			(end -0.3 -2.01)
 			(stroke
 				(width 0.12)
@@
 		)
 		(fp_line
-			(start -0.3 -1.81)
-			(end -0.3 -2.01)
+			(start 0.5 -1.2)
+			(end -1.45 -1.2)
 			(stroke
 				(width 0.12)
@@
 		)
 		(fp_line
-			(start -0.3 -1.91)
-			(end -0.6 -1.91)
+			(start 0.9 1.8)
+			(end 1.1 1.8)
 			(stroke
 				(width 0.12)
@@
 		)
 		(fp_line
-			(start -0.3 -2.01)
-			(end -0.6 -2.01)
+			(start 0.9 2.3)
+			(end 0.9 1.8)
 			(stroke
 				(width 0.12)
@@
 		)
 		(fp_line
-			(start -0.6 -2.01)
-			(end -0.6 -1.81)
+			(start 1 2.3)
+			(end 1 1.8)
 			(stroke
 				(width 0.12)
@@
 		)
 		(fp_line
-			(start -1.11 -2.11)
-			(end -2.36 -2.11)
+			(start 1.1 1.8)
+			(end 1.1 2.3)
 			(stroke
 				(width 0.12)
@@
 		)
 		(fp_line
-			(start -1.45 2.3)
-			(end 3.45 2.3)
+			(start 1.5 -1.2)
+			(end 1.5 -1.81)
 			(stroke
 				(width 0.12)
@@
 		)
 		(fp_line
-			(start -1.45 -1.2)
-			(end -1.45 2.3)
+			(start 3.45 -1.2)
+			(end 1.5 -1.2)
 			(stroke
 				(width 0.12)
@@
 		)
 		(fp_line
-			(start -2.06 2.91)
-			(end 4.06 2.91)
+			(start 3.45 2.3)
+			(end 3.45 -1.2)
 			(stroke
 				(width 0.12)
@@
 		)
 		(fp_line
-			(start -2.06 0.8)
-			(end -1.45 0.8)
+			(start 4.06 -1.81)
+			(end -2.06 -1.81)
 			(stroke
 				(width 0.12)
@@
 		)
 		(fp_line
-			(start -2.06 -0.5)
-			(end -1.45 -0.5)
+			(start 4.06 -0.5)
+			(end 3.45 -0.5)
 			(stroke
 				(width 0.12)
@@
 		)
 		(fp_line
-			(start -2.06 -1.81)
-			(end -2.06 2.91)
+			(start 4.06 0.8)
+			(end 3.45 0.8)
 			(stroke
 				(width 0.12)
@@
 		)
 		(fp_line
-			(start -2.36 -2.11)
-			(end -2.36 -0.86)
+			(start 4.06 2.91)
+			(end 4.06 -1.81)
 			(stroke
 				(width 0.12)
@@
 		)
 		(fp_line
-			(start 4.45 3.3)
-			(end 4.45 -2.2)
+			(start -2.45 -2.2)
+			(end -2.45 3.3)
 			(stroke
 				(width 0.05)
@@
 		)
 		(fp_line
-			(start 4.45 -2.2)
-			(end -2.45 -2.2)
+			(start -2.45 3.3)
+			(end 4.45 3.3)
 			(stroke
 				(width 0.05)
@@
 		)
 		(fp_line
-			(start -2.45 3.3)
-			(end 4.45 3.3)
+			(start 4.45 -2.2)
+			(end -2.45 -2.2)
 			(stroke
 				(width 0.05)
@@
 		)
 		(fp_line
-			(start -2.45 -2.2)
-			(end -2.45 3.3)
+			(start 4.45 3.3)
+			(end 4.45 -2.2)
 			(stroke
 				(width 0.05)
@@
 		)
 		(fp_line
-			(start 3.95 2.8)
-			(end 3.95 -1.7)
+			(start -2.36 -2.11)
+			(end -2.36 -0.86)
 			(stroke
 				(width 0.1)
@@
 		)
 		(fp_line
-			(start 3.95 -1.7)
-			(end -1.95 -1.7)
+			(start -1.95 -1.7)
+			(end -1.95 2.8)
 			(stroke
 				(width 0.1)
@@
 		)
 		(fp_line
-			(start -1.11 -2.11)
-			(end -2.36 -2.11)
+			(start -1.95 2.8)
+			(end 3.95 2.8)
 			(stroke
 				(width 0.1)
@@
 		)
 		(fp_line
-			(start -1.95 2.8)
-			(end 3.95 2.8)
+			(start -1.11 -2.11)
+			(end -2.36 -2.11)
 			(stroke
 				(width 0.1)
@@
 		)
 		(fp_line
-			(start -1.95 -1.7)
-			(end -1.95 2.8)
+			(start 3.95 -1.7)
+			(end -1.95 -1.7)
 			(stroke
 				(width 0.1)
@@
 		)
 		(fp_line
-			(start -2.36 -2.11)
-			(end -2.36 -0.86)
+			(start 3.95 2.8)
+			(end 3.95 -1.7)
 			(stroke
 				(width 0.1)
@@
 		)
 		(pad "1" thru_hole roundrect
-			(at 0 0 180)
+			(at 0 0)
 			(size 1.2 1.75)
 			(drill 0.75)
@@
 			(remove_unused_layers no)
 			(roundrect_rratio 0.208333)
-			(net 22 "GND")
+			(net 19 "+BATT")
 			(pinfunction "Pin_1")
 			(pintype "passive")
 		)
 		(pad "2" thru_hole oval
-			(at 2 0 180)
+			(at 2 0)
 			(size 1.2 1.75)
 			(drill 0.75)
 			(layers "*.Cu" "*.Mask")
 			(remove_unused_layers no)
-			(net 19 "+BATT")
+			(net 22 "GND")
 			(pinfunction "Pin_2")
 			(pintype "passive")
@@
 	)
 	(gr_text "BATTERY"
-		(at 84.5 66.5 0)
+		(at 84.1 72 90)
 		(layer "F.SilkS")
 		(effects
@@
 		)
 	)
+	(gr_text "+"
+		(at 96.4 63.9 0)
+		(layer "F.SilkS")
+		(effects
+			(font
+				(size 1 1)
+				(thickness 0.2)
+				(bold yes)
+			)
+			(justify left bottom)
+		)
+	)
 	(gr_text "IR"
 		(at 105.7 66.5 0)
@@
 		)
 	)
+	(gr_text "S"
+		(at 112.6 67.6 270)
+		(layer "B.SilkS")
+		(effects
+			(font
+				(size 1 1)
+				(thickness 0.2)
+				(bold yes)
+			)
+			(justify left bottom mirror)
+		)
+	)
+	(gr_text "SERVO"
+		(at 114.2 60.7 90)
+		(layer "B.SilkS")
+		(effects
+			(font
+				(size 1 1)
+				(thickness 0.1)
+			)
+			(justify left bottom mirror)
+		)
+	)
+	(gr_text "+"
+		(at 107.3 62.6 180)
+		(layer "B.SilkS")
+		(effects
+			(font
+				(size 1 1)
+				(thickness 0.2)
+				(bold yes)
+			)
+			(justify left bottom mirror)
+		)
+	)
 	(gr_text "TankIR_HAT\nFHD 2026"
 		(at 99.3 63.5 180)
@@
 			)
 			(justify left bottom mirror)
+		)
+	)
+	(gr_text "+"
+		(at 105.8 69.8 180)
+		(layer "B.SilkS")
+		(effects
+			(font
+				(size 1 1)
+				(thickness 0.2)
+				(bold yes)
+			)
+			(justify left bottom mirror)
+		)
+	)
+	(gr_text "+"
+		(at 88.6 69.9 180)
+		(layer "B.SilkS")
+		(effects
+			(font
+				(size 1 1)
+				(thickness 0.2)
+				(bold yes)
+			)
+			(justify left bottom mirror)
