File: KiCad/TankIR_Breaker/_autosave-TankIR_Breaker.kicad_sch (KiCad schematic)
At the start: 15 parts, among them J1 VBATT, J2 TRIGGER, J3 SERVO, J4 RC, J5 APPLE, J6 SOUND, J7 IR_OUT, J8 MUZZLE, Q1 BC337, Q2 BC337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

Commit message: change
Connections:
- net +BATT: now also J1.1 (Pin_1); no longer J1.2 (Pin_2)
- net GND: now also J1.2 (Pin_2); no longer J1.1 (Pin_1)
Other:
- moved on the sheet: J1
Changed lines of the file:
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@@
 	(symbol
 		(lib_id "Connector_Generic:Conn_01x02")
-		(at 25.4 91.44 180)
-		(unit 1)
-		(exclude_from_sim no)
-		(in_bom yes)
-		(on_board yes)
-		(dnp no)
-		(fields_autoplaced yes)
+		(at 25.4 88.9 0)
+		(mirror y)
+		(unit 1)
+		(exclude_from_sim no)
+		(in_bom yes)
+		(on_board yes)
+		(dnp no)
 		(property "Reference" "J1"
-			(at 25.4 82.55 0)
+			(at 22.606 89.916 0)
 			(effects
 				(font
@@
 		)
 		(property "Value" "VBATT"
-			(at 25.4 85.09 0)
+			(at 25.908 86.106 0)
 			(effects
 				(font
@@
 		)
 		(property "Footprint" "Connector_JST:JST_PH_B2B-PH-K_1x02_P2.00mm_Vertical"
-			(at 25.4 91.44 0)
+			(at 25.4 88.9 0)
 			(effects
 				(font
@@
 		)
 		(property "Datasheet" "~"
-			(at 25.4 91.44 0)
+			(at 25.4 88.9 0)
 			(effects
 				(font
@@
 		)
 		(property "Description" "Generic connector, single row, 01x02, script generated (kicad-library-utils/schlib/autogen/connector/)"
-			(at 25.4 91.44 0)
+			(at 25.4 88.9 0)
 			(effects
 				(font
@@
 		(on_board yes)
 		(dnp no)
-		(fields_autoplaced yes)
 		(property "Reference" "J2"
-			(at 25.4 95.25 0)
+			(at 24.13 99.06 0)
 			(effects
 				(font
@@
 		)
 		(property "Value" "TRIGGER"
-			(at 25.4 97.79 0)
-			(effects
-				(font
+			(at 18.796 99.314 0)
+			(effects
+				(font
